Commit message: [user] update model to remove tilt

File: user/kxr_uav/kxr_uav_fullbody.urdf (robot description, URDF)
Before this commit: robot kxr_uav_fullbody, 41 links, 40 joints
Links:
- removed link LINK34
- removed link LINK35
- removed link LINK36
- removed link LINK37
- removed link LINK38
- removed link LINK39
- link BASE: mass 0.802232 -> 0.731166; geometry collision mesh filename=package://robot_assembler/meshes/kxr_uav/uav_backpack.STL scale=0.001000 0.001000 0.001000; collision mesh filename=package://robot_assembler/meshes/kxr_uav/uav_backpack_mount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 scale=0.001000 0.001000 0.001000
- link LINK0: mass 0.035533 -> 0.012371; geometry collision mesh filename=package://robot_assembler/meshes/mesh_BOTTOM-ARM28.dae scale=1.000000 1.000000 1.000000; collision mesh filename=package://robot_assembler/meshes/mesh_JOINT-BASE.dae scale=1.000000 1.000000 1.000000
- link LINK1: mass 0.045736 -> 0.061777; geometry collision mesh filename=package://robot_assembler/meshes/mesh_CROSS-SERVO-FRAME-A.d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 scale=1.000000 1.000000 1.000000; collision mesh filename=package://robot_assembler/meshes/mesh_CROSS-SERVO-FRAME-B.d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 scale=1.000000 1.000000 1.000000
- link LINK10: mass 0.012371 -> 0.061777; geometry collision mesh filename=package://robot_assembler/meshes/mesh_CROSS-SERVO-FRAME-A.d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 scale=1.000000 1.000000 1.000000; collision mesh filename=package://robot_assembler/meshes/mesh_CROSS-SERVO-FRAME-B.d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 scale=1.000000 1.000000 1.000000
- link LINK11: mass 0.061777 -> 0.021241; geometry collision mesh filename=package://robot_assembler/meshes/mesh_BOTTOM-ARM26.dae scale=1.000000 1.000000 1.000000; collision mesh filename=package://robot_assembler/meshes/mesh_BOTTOM-ARM38.dae scale=1.000000 1.000000 1.000000
- link LINK12: mass 0.050016 -> 0.068898; geometry collision mesh filename=package://robot_assembler/meshes/mesh_BOTTOM-SPACER.dae scale=1.000000 1.000000 1.000000; collision mesh filename=package://robot_assembler/meshes/mesh_JOINT-BASE.dae scale=1.000000 1.000000 1.000000
- link LINK13: mass 0.013908 -> 0.012371; geometry collision mesh filename=package://robot_assembler/meshes/mesh_BOTTOM-ARM28.dae scale=1.000000 1.000000 1.000000; collision mesh filename=package://robot_assembler/meshes/mesh_JOINT-BASE.dae scale=1.000000 1.000000 1.000000
- link LINK14: mass 0.013908 -> 0.061777; geometry collision mesh filename=package://robot_assembler/meshes/mesh_CROSS-SERVO-FRAME-A.d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 scale=1.000000 1.000000 1.000000; collision mesh filename=package://robot_assembler/meshes/mesh_CROSS-SERVO-FRAME-B.d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 scale=1.000000 1.000000 1.000000
- link LINK15: mass 0.012371 -> 0.050016; geometry collision mesh filename=package://robot_assembler/meshes/mesh_BOTTOM-ARM38.dae scale=1.000000 1.000000 1.000000; collision mesh filename=package://robot_assembler/meshes/mesh_JOINT-BASE.dae scale=1.000000 1.000000 1.000000
- link LINK16: mass 0.061777 -> 0.013908; geometry collision mesh filename=package://robot_assembler/meshes/mesh_FINGER.dae scale=1.000000 1.000000 1.000000; visual mesh filename=package://robot_assembler/meshes/mesh_FINGER.dae scale=1.000000 1.000000 1.000000
- link LINK17: mass 0.021241 -> 0.013908; geometry collision mesh filename=package://robot_assembler/meshes/mesh_FINGER.dae scale=1.000000 1.000000 1.000000; visual mesh filename=package://robot_assembler/meshes/mesh_FINGER.dae scale=1.000000 1.000000 1.000000
- link LINK18: mass 0.068898 -> 0.035533; geometry collision mesh filename=package://robot_assembler/meshes/mesh_JOINT-BASE.dae scale=1.000000 1.000000 1.000000; collision mesh filename=package://robot_assembler/meshes/mesh_JOINT-FRAME-A.dae scale=1.000000 1.000000 1.000000
- link LINK19: mass 0.012371 -> 0.01216; geometry collision mesh filename=package://robot_assembler/meshes/mesh_BOTTOM-ARM28.dae scale=1.000000 1.000000 1.000000; collision mesh filename=package://robot_assembler/meshes/mesh_JOINT-BASE.dae scale=1.000000 1.000000 1.000000
- link LINK2: mass 0.03987 -> 0.021241; geometry collision mesh filename=package://robot_assembler/meshes/mesh_BOTTOM-ARM26.dae scale=1.000000 1.000000 1.000000; collision mesh filename=package://robot_assembler/meshes/mesh_BOTTOM-ARM38.dae scale=1.000000 1.000000 1.000000
- link LINK20: mass 0.061777 -> 0.012371; geometry collision mesh filename=package://robot_assembler/meshes/mesh_BOTTOM-ARM28.dae scale=1.000000 1.000000 1.000000; collision mesh filename=package://robot_assembler/meshes/mesh_JOINT-BASE.dae scale=1.000000 1.000000 1.000000
- link LINK21: mass 0.050016 -> 0.061777; geometry collision mesh filename=package://robot_assembler/meshes/mesh_CROSS-SERVO-FRAME-A.d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 scale=1.000000 1.000000 1.000000; collision mesh filename=package://robot_assembler/meshes/mesh_CROSS-SERVO-FRAME-B.d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 scale=1.000000 1.000000 1.000000
- link LINK22: mass 0.013908 -> 0.025166; geometry collision mesh filename=package://robot_assembler/meshes/mesh_BOTTOM-ARM20.dae scale=1.000000 1.000000 1.000000; collision mesh filename=package://robot_assembler/meshes/mesh_BOTTOM-ARM38.dae scale=1.000000 1.000000 1.000000
- link LINK23: mass 0.013908 -> 0.055048; geometry collision mesh filename=package://robot_assembler/meshes/mesh_ANGLE-BRACKET.dae scale=1.000000 1.000000 1.000000; collision mesh filename=package://robot_assembler/meshes/mesh_ANGLE-BRACKET.dae scale=1.000000 1.000000 1.000000
- link LINK24: mass 0.035533 -> 0.061777; geometry collision mesh filename=package://robot_assembler/meshes/mesh_CROSS-SERVO-FRAME-A.d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 scale=1.000000 1.000000 1.000000; collision mesh filename=package://robot_assembler/meshes/mesh_CROSS-SERVO-FRAME-B.d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 scale=1.000000 1.000000 1.000000
- link LINK25: mass 0.01216 -> 0.045736; geometry collision mesh filename=package://robot_assembler/meshes/mesh_BOTTOM-ARM28.dae scale=1.000000 1.000000 1.000000; collision mesh filename=package://robot_assembler/meshes/mesh_BOTTOM-SPACER.dae scale=1.000000 1.000000 1.000000
- link LINK26: mass 0.012371 -> 0.03987; geometry collision mesh filename=package://robot_assembler/meshes/kxr_uav/wheel_foot.STL scale=0.001000 0.001000 0.001000; visual mesh filename=package://robot_assembler/meshes/kxr_uav/wheel_foot.STL scale=0.001000 0.001000 0.001000
- link LINK27: mass 0.061777 -> 0.012371; geometry collision mesh filename=package://robot_assembler/meshes/mesh_BOTTOM-ARM28.dae scale=1.000000 1.000000 1.000000; collision mesh filename=package://robot_assembler/meshes/mesh_JOINT-BASE.dae scale=1.000000 1.000000 1.000000
- link LINK28: mass 0.025166 -> 0.061777; geometry collision mesh filename=package://robot_assembler/meshes/mesh_CROSS-SERVO-FRAME-A.d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 scale=1.000000 1.000000 1.000000; collision mesh filename=package://robot_assembler/meshes/mesh_CROSS-SERVO-FRAME-B.d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 scale=1.000000 1.000000 1.000000
- link LINK29: mass 0.055048 -> 0.025166; geometry collision mesh filename=package://robot_assembler/meshes/mesh_BOTTOM-ARM20.dae scale=1.000000 1.000000 1.000000; collision mesh filename=package://robot_assembler/meshes/mesh_BOTTOM-ARM38.dae scale=1.000000 1.000000 1.000000
- link LINK3: mass 0.035533 -> 0.068898; geometry collision mesh filename=package://robot_assembler/meshes/mesh_BOTTOM-SPACER.dae scale=1.000000 1.000000 1.000000; collision mesh filename=package://robot_assembler/meshes/mesh_JOINT-BASE.dae scale=1.000000 1.000000 1.000000
- link LINK30: mass 0.061777 -> 0.055048; geometry collision mesh filename=package://robot_assembler/meshes/mesh_ANGLE-BRACKET.dae scale=1.000000 1.000000 1.000000; collision mesh filename=package://robot_assembler/meshes/mesh_ANGLE-BRACKET.dae scale=1.000000 1.000000 1.000000
- link LINK31: mass 0.045736 -> 0.061777; geometry collision mesh filename=package://robot_assembler/meshes/mesh_CROSS-SERVO-FRAME-A.d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 scale=1.000000 1.000000 1.000000; collision mesh filename=package://robot_assembler/meshes/mesh_CROSS-SERVO-FRAME-B.d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 scale=1.000000 1.000000 1.000000
- link LINK32: mass 0.03987 -> 0.045736; geometry collision mesh filename=package://robot_assembler/meshes/mesh_BOTTOM-ARM28.dae scale=1.000000 1.000000 1.000000; collision mesh filename=package://robot_assembler/meshes/mesh_BOTTOM-SPACER.dae scale=1.000000 1.000000 1.000000
- link LINK33: mass 0.012371 -> 0.03987; geometry collision mesh filename=package://robot_assembler/meshes/kxr_uav/wheel_foot.STL scale=0.001000 0.001000 0.001000; visual mesh filename=package://robot_assembler/meshes/kxr_uav/wheel_foot.STL scale=0.001000 0.001000 0.001000
- link LINK4: mass 0.045736 -> 0.012371; geometry collision mesh filename=package://robot_assembler/meshes/mesh_BOTTOM-ARM28.dae scale=1.000000 1.000000 1.000000; collision mesh filename=package://robot_assembler/meshes/mesh_JOINT-BASE.dae scale=1.000000 1.000000 1.000000
- link LINK5: mass 0.03987 -> 0.061777; geometry collision mesh filename=package://robot_assembler/meshes/mesh_CROSS-SERVO-FRAME-A.d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 scale=1.000000 1.000000 1.000000; collision mesh filename=package://robot_assembler/meshes/mesh_CROSS-SERVO-FRAME-B.d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 scale=1.000000 1.000000 1.000000
- link LINK6: mass 0.012371 -> 0.050016; geometry collision mesh filename=package://robot_assembler/meshes/mesh_BOTTOM-ARM38.dae scale=1.000000 1.000000 1.000000; collision mesh filename=package://robot_assembler/meshes/mesh_JOINT-BASE.dae scale=1.000000 1.000000 1.000000
- link LINK7: mass 0.061777 -> 0.013908; geometry collision mesh filename=package://robot_assembler/meshes/mesh_FINGER.dae scale=1.000000 1.000000 1.000000; visual mesh filename=package://robot_assembler/meshes/mesh_FINGER.dae scale=1.000000 1.000000 1.000000
- link LINK8: mass 0.021241 -> 0.013908; geometry collision mesh filename=package://robot_assembler/meshes/mesh_FINGER.dae scale=1.000000 1.000000 1.000000; visual mesh filename=package://robot_assembler/meshes/mesh_FINGER.dae scale=1.000000 1.000000 1.000000
- link LINK9: mass 0.068898 -> 0.012371; geometry collision mesh filename=package://robot_assembler/meshes/mesh_BOTTOM-ARM28.dae scale=1.000000 1.000000 1.000000; collision mesh filename=package://robot_assembler/meshes/mesh_JOINT-BASE.dae scale=1.000000 1.000000 1.000000
Joints:
- removed joint JOINT34
- removed joint JOINT35
- removed joint JOINT36
- removed joint JOINT37
- removed joint JOINT38
- removed joint JOINT39
- joint JOINT0: origin xyz=-0.051000 -0.094000 0.058000 rpy=1.46899367 -1.57079633 -1.46899367 -> xyz=-0.051000 -0.007250 0.059500 rpy=1.57079633 -0.00000000 -1.57079633
- joint JOINT1: origin xyz=0.000000 -0.018000 0.032500 rpy=1.03037683 -1.57079633 0.54041950 -> xyz=0.000000 0.017000 0.027500 rpy=1.32581766 1.57079633 -0.24497866
- joint JOINT10: origin xyz=-0.070000 -0.000000 -0.018000 rpy=-1.46795693 1.57079633 1.67363573 -> xyz=0.000000 -0.017000 0.027500 rpy=1.12637712 1.57079633 2.69717344
- joint JOINT11: origin xyz=-0.017000 0.000000 0.027500 rpy=-3.14159265 1.57079633 -3.14159265 -> xyz=0.000000 -0.018000 0.017000 rpy=1.57079633 0.00000000 0.00000000
- joint JOINT12: origin xyz=0.000000 -0.018000 0.017000 rpy=1.57079633 0.00000000 0.00000000 -> xyz=-0.021417 0.056671 -0.017500 rpy=1.57079633 -0.00000000 -1.50250083
- joint JOINT13: origin xyz=-0.058507 0.018640 0.000500 rpy=-0.00000000 0.00000000 1.43420534 -> xyz=-0.070000 -0.000000 -0.018000 rpy=-1.51272860 1.57079633 1.62886405
- joint JOINT14: origin xyz=-0.071768 -0.000734 0.000500 rpy=-0.00000000 0.00000000 1.43420534 -> xyz=-0.017000 0.000000 0.027500 rpy=-3.14159265 1.57079633 -3.14159265; parent LINK12 -> LINK13
- joint JOINT15: origin xyz=0.051000 -0.007250 0.059500 rpy=-1.57079633 0.00000000 -1.57079633 -> xyz=0.000000 -0.018000 0.017000 rpy=1.57079633 0.00000000 0.00000000; parent BASE -> LINK14
- joint JOINT16: origin xyz=0.000000 -0.017000 0.027500 rpy=1.12637712 1.57079633 2.69717344 -> xyz=-0.058507 0.018640 0.000500 rpy=-0.00000000 0.00000000 1.43420534
- joint JOINT17: origin xyz=0.000000 -0.018000 0.017000 rpy=1.57079633 0.00000000 0.00000000 -> xyz=-0.071768 -0.000734 0.000500 rpy=-0.00000000 0.00000000 1.43420534; parent LINK16 -> LINK15
- joint JOINT18: origin xyz=-0.021417 0.056671 -0.017500 rpy=1.57079633 -0.00000000 -1.50250083 -> xyz=0.000000 -0.007250 0.077500 rpy=-0.00000000 0.00000000 -1.57079633; parent LINK17 -> BASE
- joint JOINT19: origin xyz=-0.070000 -0.000000 -0.018000 rpy=-1.51272860 1.57079633 1.62886405 -> xyz=-0.000000 -0.018000 0.032500 rpy=1.78188966 -1.57079633 -0.21109333
- joint JOINT2: origin xyz=0.065000 -0.000000 -0.017500 rpy=2.30721689 -1.57079633 0.83437577 -> xyz=0.000000 -0.018000 0.017000 rpy=1.57079633 0.00000000 0.00000000
- joint JOINT20: origin xyz=-0.017000 0.000000 0.027500 rpy=-3.14159265 1.57079633 -3.14159265 -> xyz=0.044500 -0.010500 -0.051000 rpy=3.14159265 0.00000000 0.00000000; parent LINK19 -> BASE
- joint JOINT21: origin xyz=0.000000 -0.018000 0.017000 rpy=1.57079633 0.00000000 0.00000000 -> xyz=0.000000 0.017000 0.027500 rpy=2.48054948 1.57079633 0.90975316
- joint JOINT22: origin xyz=-0.058507 0.018640 0.000500 rpy=-0.00000000 0.00000000 1.43420534 -> xyz=0.000000 -0.018000 0.017000 rpy=1.57079633 0.00000000 0.00000000
- joint JOINT23: origin xyz=-0.071768 -0.000734 0.000500 rpy=-0.00000000 0.00000000 1.43420534 -> xyz=-0.057460 -0.007898 -0.000000 rpy=-0.00000000 -0.00000000 0.13659098; parent LINK21 -> LINK22
- joint JOINT24: origin xyz=0.000000 -0.007250 0.077500 rpy=-0.00000000 0.00000000 -1.57079633 -> xyz=-0.023500 -0.053000 -0.000500 rpy=-0.00000000 -0.00000000 1.57079633; parent BASE -> LINK23
- joint JOINT25: origin xyz=-0.000000 -0.018000 0.032500 rpy=1.78188966 -1.57079633 -0.21109333 -> xyz=-0.021000 -0.017000 -0.018000 rpy=1.57079633 0.00000000 -3.14159265
- joint JOINT26: origin xyz=0.044500 -0.010500 -0.051000 rpy=3.14159265 0.00000000 0.00000000 -> xyz=0.065000 -0.000000 0.017000 rpy=1.14099359 -1.57079633 2.00059907; parent BASE -> LINK25
- joint JOINT27: origin xyz=0.000000 0.017000 0.027500 rpy=2.48054948 1.57079633 0.90975316 -> xyz=-0.044500 -0.010500 -0.051000 rpy=3.14159265 0.00000000 -3.14159265; parent LINK26 -> BASE
- joint JOINT28: origin xyz=0.000000 -0.018000 0.017000 rpy=1.57079633 0.00000000 0.00000000 -> xyz=-0.000000 -0.017000 0.027500 rpy=-1.57079633 1.57079633 0.00000000
- joint JOINT29: origin xyz=-0.057460 -0.007898 -0.000000 rpy=-0.00000000 -0.00000000 0.13659098 -> xyz=0.000000 -0.018000 0.017000 rpy=1.57079633 0.00000000 0.00000000
- joint JOINT3: origin xyz=0.051000 -0.094000 0.058000 rpy=1.96925607 -1.57079633 1.17233659 -> xyz=-0.021417 0.056671 -0.017500 rpy=1.57079633 -0.00000000 -1.50250083; parent BASE -> LINK2
- joint JOINT30: origin xyz=-0.023500 -0.053000 -0.000500 rpy=-0.00000000 -0.00000000 1.57079633 -> xyz=-0.057460 -0.007898 -0.000000 rpy=-0.00000000 -0.00000000 0.13659098
- joint JOINT31: origin xyz=-0.021000 -0.017000 -0.018000 rpy=1.57079633 0.00000000 -3.14159265 -> xyz=-0.023500 -0.053000 -0.000500 rpy=-0.00000000 -0.00000000 1.57079633
- joint JOINT32: origin xyz=0.065000 -0.000000 0.017000 rpy=1.14099359 -1.57079633 2.00059907 -> xyz=-0.021000 -0.017000 -0.018000 rpy=1.57079633 0.00000000 -3.14159265
- joint JOINT33: origin xyz=-0.044500 -0.010500 -0.051000 rpy=3.14159265 0.00000000 -3.14159265 -> xyz=0.065000 -0.000000 0.017000 rpy=0.71573506 -1.57079633 2.42585760; parent BASE -> LINK32
- joint JOINT4: origin xyz=-0.000000 0.018000 0.032500 rpy=1.57079633 -1.57079633 3.14159265 -> xyz=-0.070000 -0.000000 -0.018000 rpy=-1.46795693 1.57079633 1.67363573
- joint JOINT5: origin xyz=0.065000 -0.000000 -0.017500 rpy=2.49245391 -1.57079633 0.64913874 -> xyz=-0.017000 0.000000 0.027500 rpy=-3.14159265 1.57079633 -3.14159265
- joint JOINT6: origin xyz=-0.051000 -0.007250 0.059500 rpy=1.57079633 -0.00000000 -1.57079633 -> xyz=0.000000 -0.018000 0.017000 rpy=1.57079633 0.00000000 0.00000000; parent BASE -> LINK5
- joint JOINT7: origin xyz=0.000000 0.017000 0.027500 rpy=1.32581766 1.57079633 -0.24497866 -> xyz=-0.058507 0.018640 0.000500 rpy=-0.00000000 0.00000000 1.43420534
- joint JOINT8: origin xyz=0.000000 -0.018000 0.017000 rpy=1.57079633 0.00000000 0.00000000 -> xyz=-0.071768 -0.000734 0.000500 rpy=-0.00000000 0.00000000 1.43420534; parent LINK7 -> LINK6
- joint JOINT9: origin xyz=-0.021417 0.056671 -0.017500 rpy=1.57079633 -0.00000000 -1.50250083 -> xyz=0.051000 -0.007250 0.059500 rpy=-1.57079633 0.00000000 -1.57079633; parent LINK8 -> BASE
