Commit message: [user] update rviz urdf

File: user/kxr_uav/kxr_uav_fullbody_fin_rviz.urdf (robot description, URDF)
Before this commit: robot kxr_uav_fullbody_fin, 35 links, 34 joints
Joints:
- removed joint JOINT18
- removed joint JOINT19
- removed joint JOINT20
- removed joint JOINT21
- removed joint JOINT22
- removed joint JOINT23
- removed joint JOINT24
- removed joint JOINT25
- removed joint JOINT26
- removed joint JOINT27
- removed joint JOINT28
- removed joint JOINT29
- removed joint JOINT30
- removed joint JOINT31
- removed joint JOINT32
- removed joint JOINT33
- added joint HEAD-NECK-P: type revolute, parent LINK18, child LINK19, origin xyz=-0.000000 -0.018000 0.032500 rpy=1.78188966 -1.57079633 -0.21109333, axis 0 0 1, limit lower=-3.14159 upper=3.14159 effort=200 velocity=40
- added joint HEAD-NECK-Y: type revolute, parent BASE, child LINK18, origin xyz=0.000000 -0.007250 0.077500 rpy=-0.00000000 0.00000000 -1.57079633, axis 0 0 1, limit lower=-3.14159 upper=3.14159 effort=200 velocity=40
- added joint LLEG-ANKLE-P: type revolute, parent LINK30, child LINK31, origin xyz=-0.023500 -0.053000 -0.000500 rpy=-0.00000000 -0.00000000 1.57079633, axis 0 0 1, limit lower=-3.14159 upper=3.14159 effort=200 velocity=40
- added joint LLEG-ANKLE-R: type revolute, parent LINK31, child LINK32, origin xyz=-0.021000 -0.017000 -0.018000 rpy=1.57079633 0.00000000 -3.14159265, axis 0 0 1, limit lower=-3.14159 upper=3.14159 effort=200 velocity=40
- added joint LLEG-ANKLE-W: type revolute, parent LINK32, child LINK33, origin xyz=0.065000 -0.000000 0.017000 rpy=0.71573506 -1.57079633 2.42585760, axis 0 0 1, limit lower=-3.14159 upper=3.14159 effort=200 velocity=40
- added joint LLEG-CROTCH-P: type revolute, parent LINK28, child LINK29, origin xyz=0.000000 -0.018000 0.017000 rpy=1.57079633 0.00000000 0.00000000, axis 0 0 1, limit lower=-3.14159 upper=3.14159 effort=200 velocity=40
- added joint LLEG-CROTCH-R: type revolute, parent LINK27, child LINK28, origin xyz=-0.000000 -0.017000 0.027500 rpy=-1.57079633 1.57079633 0.00000000, axis 0 0 1, limit lower=-3.14159 upper=3.14159 effort=200 velocity=40
- added joint LLEG-CROTCH-Y: type revolute, parent BASE, child LINK27, origin xyz=-0.044500 -0.010500 -0.051000 rpy=3.14159265 0.00000000 -3.14159265, axis 0 0 1, limit lower=-3.14159 upper=3.14159 effort=200 velocity=40
- added joint LLEG-KNEE-P: type revolute, parent LINK29, child LINK30, origin xyz=-0.057460 -0.007898 -0.000000 rpy=-0.00000000 -0.00000000 0.13659098, axis 0 0 1, limit lower=-3.14159 upper=3.14159 effort=200 velocity=40
- added joint RLEG-ANKLE-P: type revolute, parent LINK23, child LINK24, origin xyz=-0.023500 -0.053000 -0.000500 rpy=-0.00000000 -0.00000000 1.57079633, axis 0 0 1, limit lower=-3.14159 upper=3.14159 effort=200 velocity=40
- added joint RLEG-ANKLE-R: type revolute, parent LINK24, child LINK25, origin xyz=-0.021000 -0.017000 -0.018000 rpy=1.57079633 0.00000000 -3.14159265, axis 0 0 1, limit lower=-3.14159 upper=3.14159 effort=200 velocity=40
- added joint RLEG-ANKLE-W: type revolute, parent LINK25, child LINK26, origin xyz=0.065000 -0.000000 0.017000 rpy=1.14099359 -1.57079633 2.00059907, axis 0 0 1, limit lower=-3.14159 upper=3.14159 effort=200 velocity=40
- added joint RLEG-CROTCH-P: type revolute, parent LINK21, child LINK22, origin xyz=0.000000 -0.018000 0.017000 rpy=1.57079633 0.00000000 0.00000000, axis 0 0 1, limit lower=-3.14159 upper=3.14159 effort=200 velocity=40
- added joint RLEG-CROTCH-R: type revolute, parent LINK20, child LINK21, origin xyz=0.000000 0.017000 0.027500 rpy=2.48054948 1.57079633 0.90975316, axis 0 0 1, limit lower=-3.14159 upper=3.14159 effort=200 velocity=40
- added joint RLEG-CROTCH-Y: type revolute, parent BASE, child LINK20, origin xyz=0.044500 -0.010500 -0.051000 rpy=3.14159265 0.00000000 0.00000000, axis 0 0 1, limit lower=-3.14159 upper=3.14159 effort=200 velocity=40
- added joint RLEG-KNEE-P: type revolute, parent LINK22, child LINK23, origin xyz=-0.057460 -0.007898 -0.000000 rpy=-0.00000000 -0.00000000 0.13659098, axis 0 0 1, limit lower=-3.14159 upper=3.14159 effort=200 velocity=40

Commit message: [user] add floating joint and renamed link BASE to BODY

File: user/kxr_uav/kxr_uav_fullbody_fin_rviz.urdf (robot description, URDF)
Before this commit: robot kxr_uav_fullbody_fin, 35 links, 34 joints
Links:
- added link BODY, mass 0.731166; collision mesh filename=package://robot_assembler/meshes/kxr_uav/uav_backpack.STL scale=0.001000 0.001000 0.001000; collision mesh filename=package://robot_assembler/meshes/kxr_uav/uav_backpack_mount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 scale=0.001000 0.001000 0.001000
- link BASE: mass 0.731166 -> None; geometry 
Joints:
- added joint BASE_JOINT: type floating, parent BASE, child BODY
- joint HEAD-NECK-Y: parent BASE -> BODY
- joint LARM-SHOULDER-P: parent BASE -> BODY
- joint LLEG-CROTCH-Y: parent BASE -> BODY
- joint RARM-SHOULDER-P: parent BASE -> BODY
- joint RLEG-CROTCH-Y: parent BASE -> BODY
