Commit message: [user] update kxr_uav model and mesh(may include mistake)

File: user/kxr_uav/kxr_uav_fullbody_fin_nobackpack.urdf (robot description, URDF)
Before this commit: robot kxr_uav_fullbody_fin_nobackpack, 35 links, 34 joints
Links:
- link LINK19: mass 0.01216 -> 0.05886; geometry collision mesh filename=package://robot_assembler/meshes/kxr_uav/marker_head.STL scale=0.001000 0.001000 0.001000; collision mesh filename=package://robot_assembler/meshes/mesh_BOTTOM-ARM28.dae scale=1.000000 1.000000 1.000000
