Commit message: []

File: sample/kxr_auv/kxr_auv_fullbody_initial.urdf (robot description, URDF)
Before this commit: robot kxr_auv_fullbody_initial, 26 links, 25 joints
Joints:
- joint head-neck-p: origin xyz=-0.010500 -0.018000 0.032500 rpy=1.34156439 -1.57079633 0.22923193 -> xyz=-0.010500 -0.018000 0.032500 rpy=1.57079633 -1.57079633 0.00000000
- joint head-neck-y: origin xyz=0.000000 -0.007250 0.077500 rpy=-0.00000000 0.00000000 -1.57079633 -> xyz=-0.007250 0.000000 0.077500 rpy=-0.00000000 -0.00000000 3.14159265
- joint larm-elbow-p: origin xyz=0.017500 -0.000000 0.025500 rpy=1.04133636 1.57079633 1.04133636 -> xyz=0.017500 -0.000000 0.025500 rpy=0.55897139 1.57079633 0.55897139
- joint larm-gripper-r: origin xyz=-0.055500 -0.018000 -0.018000 rpy=2.04519621 -1.57079633 -0.47439988 -> xyz=-0.055500 -0.018000 -0.018000 rpy=2.24553727 -1.57079633 -0.67474094
- joint larm-gripper2-r: origin xyz=-0.066000 -0.018000 -0.039000 rpy=2.04519621 -1.57079633 -0.47439988 -> xyz=-0.066000 -0.018000 -0.039000 rpy=2.24553727 -1.57079633 -0.67474094
- joint larm-shoulder-p: origin xyz=-0.051000 -0.007250 0.059500 rpy=1.57079633 -0.00000000 -1.57079633 -> xyz=-0.007250 0.051000 0.059500 rpy=1.57079633 -0.00000000 3.14159265
- joint larm-shoulder-r: origin xyz=-0.012374 0.012374 0.025500 rpy=0.69865982 1.57079633 3.05485431 -> xyz=-0.012374 0.012374 0.025500 rpy=1.23755203 1.57079633 -2.68943879
- joint lleg-crotch-r: origin xyz=-0.023500 -0.017000 -0.036000 rpy=-1.34608516 -1.57079633 -0.22471117 -> xyz=-0.017000 0.023500 -0.036000 rpy=-1.33234575 -1.57079633 -1.80924691
- joint rarm-elbow-p: origin xyz=0.017500 -0.000000 0.025500 rpy=1.20268268 1.57079633 1.20268268 -> xyz=0.017500 0.000000 0.025500 rpy=-0.39121759 1.57079633 -0.39121759
- joint rarm-gripper-r: origin xyz=-0.055500 -0.018000 -0.018000 rpy=2.16797298 -1.57079633 -0.59717666 -> xyz=-0.055500 -0.018000 -0.018000 rpy=2.24131788 -1.57079633 -0.67052156
- joint rarm-gripper2-r: origin xyz=-0.066000 -0.018000 -0.039000 rpy=2.16797298 -1.57079633 -0.59717666 -> xyz=-0.066000 -0.018000 -0.039000 rpy=2.24131788 -1.57079633 -0.67052156
- joint rarm-shoulder-p: origin xyz=0.051000 -0.007250 0.059500 rpy=-1.57079633 0.00000000 -1.57079633 -> xyz=-0.007250 -0.051000 0.059500 rpy=-1.57079633 0.00000000 3.14159265
- joint rarm-shoulder-r: origin xyz=0.012374 0.012374 0.025500 rpy=1.37669023 1.57079633 2.16208839 -> xyz=0.012374 0.012374 0.025500 rpy=0.96470161 1.57079633 1.75009977
- joint rleg-crotch-r: origin xyz=0.023500 -0.017000 -0.036000 rpy=-1.34608516 -1.57079633 -0.22471117 -> xyz=-0.017000 -0.023500 -0.036000 rpy=-1.33234575 -1.57079633 -1.80924691
